File: chirp-ble.brd (EAGLE design)
At the start: 122.8 x 17.5 mm, 29 parts, among them Q1 ILCX13-FF5F18-32.0000, U1 NRF52832, Y1 ABS07-32.768KHZ-7

Commit message: Fully routed
Parts:
- added TP4: TPB1,27, testpad:B1,27
- Q1: value ILCX13-FF5F18-32.0000 -> ILCX13-FF5F18-32.0000
- S1: value SWITCH-MOMENTARY-2-SMD-1101NE -> SWITCH-MOMENTARY-2SMD-1101NE
- moved SWD 3.86 mm to (54.6, 12.1)
- moved BAT1 3.81 mm to (44.2, 8.13)
- moved LED1 3.29 mm to (44.1, 9.16), turned to 0 degrees
- moved C9 3.21 mm to (29.8, 10.6), turned to 90 degrees
- moved L1 2.67 mm to (28.2, 11.2)
- moved S1 2.40 mm to (47.2, 9.14), turned to 270 degrees
- moved TP2 2.01 mm to (51.0, 1.56)
- moved R3 1.59 mm to (44.1, 12.6)
- moved C7 1.56 mm to (27.8, 7.57)
- moved C8 1.56 mm to (27.8, 8.65)
- moved C2 0.72 mm to (39.9, 14.4)
- moved C13 0.25 mm to (41.5, 11.2), turned to 0 degrees
- moved C12 0.19 mm to (41.5, 6.10), turned to 180 degrees
Connections:
- net LED renamed LED_K
- removed net G1: Q1.4
- removed net G2: Q1.2
- removed net N$14: SWD.SWO
- removed net N$5: SWD.VTREF
- removed net VSS: U1.GND
- new net LED_A: LED1.A, U1.12
- net BTN: now also S1.1; no longer S1.P$1
- net GND: now also Q1.2, Q1.4, S1.2, TP4.TP, U1.GND; no longer S1.P$2
- net VCC: now also BAT1.PWR@2, SWD.VTREF; no longer LED1.A
Routing:
- net SWDCLK: track 1.54 -> 25.6 mm, vias 0 -> 1
- net SWDIO: track 2.47 -> 24.1 mm, vias 0 -> 1
- net NRST: track 6.82 -> 25.8 mm, vias 0 -> 2
- net VCC: track 14.0 -> 29.7 mm, vias 2 -> 3
- net BTN: track 1.62 -> 15.4 mm, vias 1 -> 2
- net LED_K: track 1.44 -> 12.8 mm, vias 1 -> 2
- net GND: track 0.90 -> 10.5 mm, vias 15 -> 24
- net LED_A: track 0.00 -> 8.99 mm
- net ANT: track 6.76 -> 3.67 mm
- net V_CAP: track 34.0 -> 36.8 mm
- net N$4: track 1.22 -> 4.01 mm
- net N$6: track 0.00 -> 1.90 mm
- net Y1_P: track 4.02 -> 5.84 mm
- net N$12: track 2.77 -> 4.39 mm
- net Y1_M: track 4.08 -> 5.59 mm
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Other:
- board text removed: "ISP"

Commit message: DRC and ERC
Parts:
- moved C8 0.10 mm to (27.8, 8.75)
Routing:
- net VCC: track 29.7 -> 28.0 mm
- net GND: vias 24 -> 28
