File: chirp-ble.brd (EAGLE design)
At the start: 122.8 x 17.5 mm, 30 parts, among them Q1 ILCX13-FF5F18-32.0000, U1 NRF52832, Y1 ABS07-32.768KHZ-7

Commit message: Spike
Parts:
- Q1: value ILCX13-FF5F18-32.0000 -> YIC 32.00M-SMDXT324
- Y1: value ABS07-32.768KHZ-7 -> 32.768K-CFPX217
- moved R1 17.0 mm to (46.2, 18.5)
Routing:
- net CLK_OUT: track 19.2 -> 0.00 mm
- net V_CAP: track 36.8 -> 26.6 mm
- net CAP_V: track 18.4 -> 11.0 mm
- net GND: track 10.5 -> 9.34 mm

Commit message: Changed min drill size to 0.4mm
Parts:
- moved R1 21.7 mm to (30.1, 3.97)
- moved TP4 20.3 mm to (33.3, 1.80)
- moved TP1 19.8 mm to (15.6, 1.93)
- moved C4 18.3 mm to (25.8, 2.88)
- moved R2 18.3 mm to (23.5, 2.88)
- moved C13 18.3 mm to (23.2, 11.4)
- moved C6 18.3 mm to (18.4, 4.31)
- moved ANTENNA 18.3 mm to (6.10, 15.0)
- moved C11 18.3 mm to (7.96, 4.66)
- moved C2 18.3 mm to (21.6, 14.6)
- moved C3 18.3 mm to (14.2, 4.66)
- moved C7 18.3 mm to (9.48, 7.82)
- moved C8 18.3 mm to (9.48, 9.00)
- moved C9 18.3 mm to (11.6, 10.8)
- moved L1 18.3 mm to (9.87, 11.5)
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Connections:
- net CLK_OUT: now also U1.6; no longer U1.38
Routing:
- net CLK_OUT: track 0.00 -> 14.4 mm, vias 0 -> 2
- net CAP_V: track 11.0 -> 19.5 mm
- net V_CAP: track 26.6 -> 32.8 mm
- net Y1_P: track 5.84 -> 6.78 mm
- net VCC: track 28.0 -> 28.8 mm
- net GND: vias 28 -> 70
